Commit message: 와플파이 2개 위치 생성
한 것
1. 와플 파이 2개를 맵에 맞게 넣음
할 것
1. NAV 동작 확인해보기
2. 이를 넣어보기

File: ws/src/mars_plan/urdf/turtlebot3_waffle_pi.urdf (robot description, URDF)
Before this commit: robot turtlebot3_waffle, 13 links, 12 joints
Links:
- removed link camera_depth_frame
- removed link camera_depth_optical_frame
- link camera_link: geometry collision box size=0.015 0.030 0.027
Joints:
- removed joint camera_depth_joint
- removed joint camera_depth_optical_joint
- joint camera_joint: origin xyz=0.064 -0.065 0.094 rpy=0 0 0 -> xyz=0.073 -0.011 0.084 rpy=0 0 0
- joint camera_rgb_joint: origin xyz=0.005 0.018 0.013 rpy=0 0 0 -> xyz=0.003 0.011 0.009 rpy=0 0 0
