Commit message: 추가공부
한것:
1. ws_new 신규 생성
1-1 맵 신규 생성
1-2 imu 문제 해결
2. ws 맵 변경해서, 기존 mar.map으로 다시 바꿔야 함.

File: ws_new/src/car_track/urdf/gazebo.xacro (robot description, xacro)
@@ -19,3 +19,30 @@
         </plugin>
     </gazebo>
+    <!-- IMU SENSOR 추가 -->
+    <gazebo reference="imu_link">
+        <sensor type="imu" name="imu_sensor">
+            <update_rate>100</update_rate>
+            <imu>
+                <angular_velocity>
+                    <noise type="gaussian">
+                        <mean>0.0</mean>
+                        <stddev>0.02</stddev>
+                    </noise>
+                </angular_velocity>
+                <linear_acceleration>
+                    <noise type="gaussian">
+                        <mean>0.0</mean>
+                        <stddev>0.02</stddev>
+                    </noise>
+                </linear_acceleration>
+            </imu>
+            <plugin name="imu_plugin" filename="libgazebo_ros_imu_sensor.so">
+                <ros>
+                    <argument>~/out:=imu/data</argument>
+                </ros>
+                <output_type>sensor_msgs/Imu</output_type>
+                <frame_name>imu_link</frame_name>
+            </plugin>
+        </sensor>
+    </gazebo>
 </robot>

File: ws_new/src/car_track/urdf/lidar.xacro (robot description, xacro)
@@ -1,3 +1,36 @@
 <?xml version="1.0"?>
+<robot xmlns:xacro="http://www.ros.org/wiki/xacro">
+    <gazebo reference="laser_frame">
+        <material>Gazebo/Red</material>
+        <sensor name="laser" type="ray">
+            <pose>0 0 0 0 0 0</pose>
+            <visualize>true</visualize>
+            <update_rate>10</update_rate>
+            <ray>
+                <scan>
+                    <horizontal>
+                        <samples>360</samples>  <!-- 샘플 개수 증가 -->
+                        <resolution>1</resolution> <!-- 해상도 추가 -->
+                        <min_angle>-3.14</min_angle>
+                        <max_angle>3.14</max_angle>
+                    </horizontal>
+                </scan>
+                <range>
+                    <min>0.1</min>  <!-- 더 작은 물체도 감지 가능 -->
+                    <max>5</max>   <!-- 최대 거리 증가 -->
+                </range>
+            </ray>
+            <plugin name="laser_controller" filename="libgazebo_ros_ray_sensor.so">
+                <ros>
+                    <argument>~/out:=scan</argument>
+                </ros>
+                <output_type>sensor_msgs/LaserScan</output_type>
+                <frame_name>laser_frame</frame_name>
+            </plugin>
+        </sensor>
+    </gazebo>
+</robot>
+<!-- old_ver : 삼각형 라이다 형태여서 밑에서 원으로 수정 -->
+<!-- <?xml version="1.0"?>
 <robot xmlns:xacro="http://www.ros.org/wiki/xacro">
     <gazebo reference="laser_frame">
@@ -29,3 +62,3 @@
         </sensor>
     </gazebo>
-</robot>
+</robot> -->

File: ws_new/src/car_track/urdf/robot_4.xacro (robot description, xacro)
@@ -144,4 +144,28 @@
         </collision>
     </link>
+    <!-- IMU LINK 추가 -->
+    <joint name="imu_joint" type="fixed">
+        <parent link="base_link"/>  <!-- IMU는 로봇 본체에 부착 -->
+        <child link="imu_link"/>
+        <origin xyz="0.05 0 0.1" rpy="0 0 0"/> <!-- IMU 위치 조정 -->
+    </joint>
+    <link name="imu_link">
+        <visual>
+            <geometry>
+                <box size="0.02 0.02 0.02"/>  <!-- IMU 크기 -->
+            </geometry>
+            <material name="blue"/>
+        </visual>
+        <collision>
+            <geometry>
+                <box size="0.02 0.02 0.02"/>
+            </geometry>
+        </collision>
+        <inertial>
+            <mass value="0.05"/>
+            <origin xyz="0 0 0" rpy="0 0 0"/>
+            <inertia ixx="1.0e-5" iyy="1.0e-5" izz="1.0e-5"/>
+        </inertial>
+    </link>
     <!-- GAZEBO -->
     <xacro:include filename="gazebo.xacro"/>

Commit message: base_footprint 추가
한 것
1. nav2에 필요한 base_footprint 추가함

File: ws_new/src/car_track/urdf/gazebo.xacro (robot description, xacro)
@@ -12,9 +12,10 @@
             <max_wheel_acceleration>10.0</max_wheel_acceleration>
             <!-- Output -->
-            <odometry_frame>odom</odometry_frame>
-            <robot_base_frame>base_link</robot_base_frame>
             <publish_odom>true</publish_odom>
             <publish_odom_tf>true</publish_odom_tf>
-            <publish_wheel_tf>true</publish_wheel_tf>
+            <publish_wheel_tf>false</publish_wheel_tf>
+            <odometry_topic>odom</odometry_topic>
+            <odometry_frame>odom</odometry_frame>
+            <robot_base_frame>base_footprint</robot_base_frame>
         </plugin>
     </gazebo>

File: ws_new/src/car_track/urdf/robot_4.xacro (robot description, xacro)
@@ -16,4 +16,10 @@
         <color rgba="1 0 0 1"/>
     </material>
+  <link name="base_footprint"/>
+  <joint name="base_joint" type="fixed">
+    <parent link="base_footprint"/>
+    <child link="base_link" />
+    <origin xyz="0 0 0.010" rpy="0 0 0"/>
+  </joint>
     <!-- BASE LINK -->
     <link name="base_link">
